Commit message: Added urdf file

File: Simulation-Development/workspace/src/robot_sim/urdf/robot.urdf (robot description, URDF)
Before this commit: robot infinity_robot, 4 links, 3 joints
Links:
- link base_link: mass None -> 5.0
- link left_wheel: mass None -> 0.5
- link right_wheel: mass None -> 0.5
Joints:
- joint left_wheel_joint: type fixed -> continuous
- joint right_wheel_joint: type fixed -> continuous
